Commit message: added robot descriptions

File: urdf2model/robot_descriptions/kortex_description/urdf/JACO3_URDF_V10.urdf (robot description, URDF)
Before this commit: robot JACO3_URDF_V10, 9 links, 8 joints
Links:
- removed link Wrist1_Link
- removed link Wrist2_Link
- added link SphericalWrist1_Link, mass 0.678106; collision mesh filename=package://kortex_description/meshes/SphericalWrist1_Link.STL; visual mesh filename=package://kortex_description/meshes/SphericalWrist1_Link.STL
- added link SphericalWrist2_Link, mass 0.678106; collision mesh filename=package://kortex_description/meshes/SphericalWrist2_Link.STL; visual mesh filename=package://kortex_description/meshes/SphericalWrist2_Link.STL
- link Bracelet_Link: mass 0.31408 -> 0.500657; geometry collision mesh filename=package://kortex_description/meshes/Bracelet_Link.STL; visual mesh filename=package://kortex_description/meshes/Bracelet_Link.STL
- link EndEffector_Link: geometry collision mesh filename=package://kortex_description/meshes/EndEffector_Link.STL; visual mesh filename=package://kortex_description/meshes/EndEffector_Link.STL
- link ForeArm_Link: mass 0.895 -> 0.930287; geometry collision mesh filename=package://kortex_description/meshes/ForeArm_Link.STL; visual mesh filename=package://kortex_description/meshes/ForeArm_Link.STL
- link HalfArm1_Link: mass 1.106 -> 1.163667; geometry collision mesh filename=package://kortex_description/meshes/HalfArm1_Link.STL; visual mesh filename=package://kortex_description/meshes/HalfArm1_Link.STL
- link HalfArm2_Link: mass 1.106 -> 1.16366; geometry collision mesh filename=package://kortex_description/meshes/HalfArm2_Link.STL; visual mesh filename=package://kortex_description/meshes/HalfArm2_Link.STL
- link Shoulder_Link: mass 2.009 -> 1.377353; geometry collision mesh filename=package://kortex_description/meshes/Shoulder_Link.STL; visual mesh filename=package://kortex_description/meshes/Shoulder_Link.STL
- link base_link: mass 1.661 -> 1.697353; geometry collision mesh filename=package://kortex_description/meshes/base_link.STL; visual mesh filename=package://kortex_description/meshes/base_link.STL
Joints:
- removed joint Endeffector
- added joint EndEffector: type fixed, parent Bracelet_Link, child EndEffector_Link, origin xyz=0 0 -0.061525 rpy=3.1416 1.0815E-32 0, axis 0 0 0
- joint Actuator1: origin xyz=0 0 0.15643 rpy=3.1416 0 0 -> xyz=6.1995E-05 0 0.15643 rpy=-3.1416 3.2891E-18 1.9637E-50
- joint Actuator2: limit lower=-2.2000 upper=2.2000 effort=39 velocity=0.8727 -> lower=-2.2 upper=2.2 effort=39 velocity=0.8727; origin xyz=0 0.005375 -0.12838 rpy=1.5708 0 0 -> xyz=0 0.005375 -0.12838 rpy=1.5708 2.4106E-17 3.1919E-16
- joint Actuator3: origin xyz=0 -0.21038 -0.006375 rpy=-1.5708 0 0 -> xyz=0 -0.21038 -0.006375 rpy=-1.5708 9.8608E-32 -2.7983E-16
- joint Actuator4: origin xyz=0 0.006375 -0.21038 rpy=1.5708 0 0 -> xyz=0 0.006375 -0.21038 rpy=1.5708 3.0688E-17 -6.9389E-18
- joint Actuator5: child Wrist1_Link -> SphericalWrist1_Link; origin xyz=0 -0.20843 -0.006375 rpy=-1.5708 0 0 -> xyz=0 -0.20843 -0.006375 rpy=-1.5708 1.497E-17 7.6501E-17
- joint Actuator6: child Wrist2_Link -> SphericalWrist2_Link; limit lower=-2.0500 upper=2.0500 effort=9 velocity=0.8727 -> lower=-2.05 upper=2.05 effort=9 velocity=0.8727; origin xyz=0 0.00017505 -0.10593 rpy=1.5708 0 0 -> xyz=0 0.00017505 -0.10593 rpy=1.5708 3.3255E-17 -8.0962E-15; parent Wrist1_Link -> SphericalWrist1_Link
- joint Actuator7: origin xyz=0 -0.10593 -0.00017505 rpy=-1.5708 0 0 -> xyz=0 -0.10593 -0.00017505 rpy=-1.5708 -2.3419E-17 1.52E-17; parent Wrist2_Link -> SphericalWrist2_Link
