Commit message: update

File: urdf2model/models/xarm6/xarm6.urdf (robot description, URDF)
Before this commit: robot xarm6, 10 links, 9 joints
Links:
- link link1: mass 2.382 -> 2.177
- link link2: mass 2.267 -> 2.011
- link link3: mass 1.875 -> 1.725
- link link4: mass 1.319 -> 1.211
- link link5: mass 1.34 -> 1.206
